File: usb_to_gpib.sch (KiCad schematic (older format))
At the start: 36 parts, among them P1 CONN_12X2, P2 CONN_6, SW1 SW_PUSH, U2 FT232RL, U3 PIC18F4520, X1 CRYSTAL

Commit message: Initial commit of revC changes.
Parts:
- removed R10, R11, R12, R13, R14, R15, R16, R17, R3, R4, R5, R6, R7, R8, R9: 1k, symbol R
- removed R18, R19: 270, symbol R
- removed U2: FT232RL, symbol FT232RL
- added C10, C12: 47pF, ~, symbol C
- added C13: 4.7nF, ~, symbol C
- added C5, C9: 100nF, ~, symbol C
- added C8: 10nF, symbol C
- added RP1: 27ohm, ~, symbol R_PACK2
- added RP2: 270ohm, ~, symbol R_PACK2
- added U2: SN75160B, MODULE, symbol SN75160B
- added U3: SN75162B, MODULE, symbol SN75162B
- added U4: FT230X, MODULE, symbol FT230X
- C11: renamed from C3; value 100nF -> 10nF
- C7: renamed from C5; value 10nF -> 100nF
- R2: value 1k -> 1M; footprint (none) -> ~
- renumbered C6 to C2, C7 to C3, C2 to C4, C4 to C6, D2 to D1, D1 to D2, U3 to U1
Connections:
- net labels added: 3V3OUT, ATN, DAV, DC, DIO1, DIO2, DIO3, DIO4, DIO5, DIO6, DIO7, DIO8, EOI, ERROR_LED, FTDI_RXI, FTDI_TXO, G_ATN, G_DAV, G_DIO1, G_DIO2, G_DIO3, G_DIO4, G_DIO5, G_DIO6, G_DIO7, G_DIO8, G_EOI, G_IFC, G_NDAC, G_NRFD, G_REN, G_SRQ, IFC, NDAC, NRFD, PE, REN, SC, SRQ, TE, USB_D+, USB_D-
- wire segments 178 -> 201
- no-connect marks 1 -> 24
Other:
- moved on the sheet: C11, C4, C6, C7, D1, D2, L1, P1
