File: usb_to_gpib.sch (KiCad schematic (older format))
At the start: 29 parts, among them P1 CONN_12X2, P2 CONN_6, SW1 SW_PUSH, U1 PIC18F4520, U2 SN75160B, U3 SN75162B, U4 FT230X, X1 CRYSTAL

Commit message: Revision 4 commit
Features tx and rx LEDs on the FT230X, hardware flow lines are wired up, and a few unused dio lines are wired to ground to provide a way to distinguish between hardware revisions in software here forward.
Parts:
- added D3, D4: LED, symbol LED
- added P3, P4: CONN_1, symbol CONN_1
- added RP3: 270ohm, ~, symbol R_PACK2
Connections:
- net labels added: FTDI_CTS, FTDI_RTS, RX_LED, TX_LED
- wire segments 201 -> 228
- no-connect marks 24 -> 14
